File: kicad/_autosave-rgb.sch (KiCad schematic (older format))
At the start: 36 parts, among them J1 1935776, J2 102-6164-ND, J3 102-6164-ND, J4 Conn_01x04, J5 Conn_01x02, Q1 Si4101DY, Q2 DMG9926USD, Q3 DMG9926USD, Q4 DMG9926USD, Q5 DMG9926USD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

Commit message: rev1
Parts:
- J4: footprint Connector_PinHeader_2.54mm:PinHeader_1x03_P2.54mm_Vertical -> Connector_PinHeader_2.54mm:PinHeader_1x01_P2.54mm_Vertical
Connections:
- net DRAIN_1: now also Q2.D2; no longer Q2.D1 (D2)
- net DRAIN_2: now also Q2.D1 (D2); no longer Q2.D2
- net GND: now also Q2.S1 (S2), Q2.S2; no longer Q2.S1 (S2), Q2.S2
- net PWM_1: now also Q2.G2; no longer Q2.G1 (G2)
- net PWM_2: now also Q2.G1 (G2); no longer Q2.G2
- net PWR_EN: now also SW1.1; no longer SW1.2
- net at R3.1: now also SW1.2; no longer SW1.1
Changed lines of the file:
@@
 F 0 "J4" H 9805 4303 50  0000 C CNN
 F 1 "Conn_01x04" H 9723 4069 50  0001 C CNN
-F 2 "Connector_PinHeader_2.54mm:PinHeader_1x03_P2.54mm_Vertical" H 9805 4403 50  0001 C CNN
+F 2 "Connector_PinHeader_2.54mm:PinHeader_1x01_P2.54mm_Vertical" H 9805 4403 50  0001 C CNN
 F 3 "~" H 9805 4403 50  0001 C CNN
 	1    9805 4403
@@
 $Comp
 L mosfet:DMG9926USD Q2
-U 1 1 5FE90B41
+U 2 1 5FE90B41
 P 6655 2803
 F 0 "Q2" H 6780 2803 50  0000 L CNN
@@
 F 2 "rgb_footprints:DMG9926USD_Handsolder" H 6555 2303 50  0001 C CNN
 F 3 "https://www.diodes.com/assets/Datasheets/ds31757.pdf" H 6080 2963 50  0001 C CNN
-	1    6655 2803
+	2    6655 2803
 	1    0    0    -1
 $EndComp
@@
 $Comp
 L mosfet:DMG9926USD Q2
-U 2 1 60225873
+U 1 1 60225873
 P 8105 2803
 F 0 "Q2" H 8230 2803 50  0000 L CNN
@@
 F 2 "rgb_footprints:DMG9926USD_Handsolder" H 8005 2303 50  0001 C CNN
 F 3 "https://www.diodes.com/assets/Datasheets/ds31757.pdf" H 7530 2963 50  0001 C CNN
-	2    8105 2803
+	1    8105 2803
 	1    0    0    -1
 $EndComp
@@
 F 3 "https://www.te.com/commerce/DocumentDelivery/DDEController?Action=srchrtrv&DocNm=1825910&DocType=Customer+Drawing&DocLang=English" H 7300 1500 50  0001 C CNN
 	1    7300 1300
-	1    0    0    -1
+	-1   0    0    -1
 $EndComp
 $Comp
@@
 	1700 950  2050 950
 $Comp
-L power:PWR_FLAG #FLG?
+L power:PWR_FLAG #FLG0101
 U 1 1 6099FCA9
 P 1750 850
-F 0 "#FLG?" H 1750 925 50  0001 C CNN
+F 0 "#FLG0101" H 1750 925 50  0001 C CNN
 F 1 "PWR_FLAG" H 1750 1023 50  0001 C CNN
 F 2 "" H 1750 850 50  0001 C CNN
