File: kicad/rgb.kicad_pcb (KiCad board)
At the start: 2 copper layers, 74 x 44 mm, 28 parts, among them J1 1935776, J2 102-6164-ND, J3 102-6164-ND, J4 Conn_01x04, J5 Conn_01x02, Q1 DMG9926USD, Q2 DMG9926USD, Q3 DMG9926USD, Q4 DMG9926USD, SW1 450-1642-ND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

Commit message: rev0
Other:
- rule pad_to_mask_clearance: 0.05 -> 0
- board text added: "JLCJLCJLCJLC"

Commit message: rev1
Parts:
- removed the C1 at (182.4, 80.8)
- added Q5: DMG9926USD, rgb_footprints:DMG9926USD_Handsolder, B.Cu at (169.6, 67.0)
- added R10: 50 kΩ, Resistor_SMD:R_0805_2012Metric_Pad1.20x1.40mm_HandSolder, F.Cu at (228.4, 116.0)
- added R11: 50 kΩ, Resistor_SMD:R_0805_2012Metric_Pad1.20x1.40mm_HandSolder, F.Cu at (221.3, 119.8)
- added R12: 50 kΩ, Resistor_SMD:R_0805_2012Metric_Pad1.20x1.40mm_HandSolder, F.Cu at (226.1, 119.8)
- added R13: 50 kΩ, Resistor_SMD:R_0805_2012Metric_Pad1.20x1.40mm_HandSolder, F.Cu at (233.1, 116.0)
- added R6: 50 kΩ, Resistor_SMD:R_0805_2012Metric_Pad1.20x1.40mm_HandSolder, F.Cu at (202.3, 119.8)
- added R7: 50 kΩ, Resistor_SMD:R_0805_2012Metric_Pad1.20x1.40mm_HandSolder, F.Cu at (207.1, 119.8)
- added R8: 50 kΩ, Resistor_SMD:R_0805_2012Metric_Pad1.20x1.40mm_HandSolder, F.Cu at (211.8, 119.8)
- added R9: 50 kΩ, Resistor_SMD:R_0805_2012Metric_Pad1.20x1.40mm_HandSolder, F.Cu at (216.6, 119.8)
- Q1: value DMG9926USD -> Si4101DY; footprint rgb_footprints:DMG9926USD_Handsolder -> rgb_footprints:Si4101DY; moved to F.Cu
- R1: value 0.005 -> 5 mΩ
- R2: value 10k -> 10 kΩ
- R3: value 110k -> 110 kΩ
- moved Q1 45.8 mm to (214.2, 78.2), turned to 90 degrees
- moved Q3 30.2 mm to (160.2, 90.1), turned to 270 degrees
- moved Q4 10.1 mm to (179.7, 67.0)
- moved Q2 9.85 mm to (170.1, 90.3)
- moved J3 0.35 mm to (187.4, 62.0)
- renumbered C3 to C1, C4 to C2
Connections:
- J4 pad 1: GND -> /RESET
- J4 pad 2: /RESET -> (no net)
- J4 pad 3: +5V -> (no net)
- Q2 pad D1: /DRAIN_4 -> /DRAIN_1
- Q2 pad D2: /DRAIN_3 -> /DRAIN_2
- Q2 pad G1: /PWM_4 -> /PWM_1
- Q2 pad G2: /PWM_3 -> /PWM_2
- Q3 pad D1: /DRAIN_5 -> /DRAIN_4
- Q3 pad D2: /DRAIN_6 -> /DRAIN_3
- Q3 pad G1: /PWM_5 -> /PWM_4
- Q3 pad G2: /PWM_6 -> /PWM_3
- Q4 pad D1: /DRAIN_7 -> /DRAIN_5
- Q4 pad D2: /DRAIN_8 -> /DRAIN_6
- Q4 pad G1: /PWM_7 -> /PWM_5
- Q4 pad G2: /PWM_8 -> /PWM_6
- R1 pad 1: Net-(F1-Pad1) -> Net-(Q1-Pad3)
- U1 pad 1: Net-(F1-Pad1) -> Net-(Q1-Pad3)
Routing:
- net Net-(Q1-Pad3): track 0.00 -> 7.21 mm
- net Net-(F1-Pad1): track 7.21 -> 0.00 mm
- net GND: vias 13 -> 11
- net /DRAIN_8: vias 0 -> 2

Commit message: rev1
Parts:
- J4: footprint Connector_PinHeader_2.54mm:PinHeader_1x03_P2.54mm_Vertical -> Connector_PinHeader_2.54mm:PinHeader_1x01_P2.54mm_Vertical
- moved R13 79.5 mm to (165.7, 73.8), turned to 270 degrees
- moved R12 73.9 mm to (168.3, 73.8), turned to 270 degrees
- moved R10 69.2 mm to (173.6, 73.7), turned to 270 degrees
- moved R11 68.3 mm to (170.9, 73.8), turned to 270 degrees
- moved R9 65.4 mm to (160.1, 86.8), turned to 90 degrees
- moved R8 59.2 mm to (162.7, 86.8), turned to 90 degrees
- moved R7 53.3 mm to (165.2, 86.8), turned to 90 degrees
- moved R6 47.8 mm to (167.8, 86.8), turned to 90 degrees
- moved R2 33.0 mm to (194.4, 74.9)
- moved Q1 23.0 mm to (191.3, 80.2), turned to 0 degrees
- moved J4 20.4 mm to (150.6, 97.6), turned to 0 degrees
- moved U1 7.36 mm to (191.4, 74.8), turned to 90 degrees
- moved R1 7.23 mm to (185.3, 80.1), turned to 180 degrees
- moved J1 5.57 mm to (189.2, 87.4), turned to 180 degrees
- moved F1 1.78 mm to (193.9, 85.5)
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Connections:
- Q1 pad D: (no net) -> Net-(F1-Pad1)
- Q1 pad G: (no net) -> GND
- Q1 pad S: (no net) -> Net-(Q1-PadS)
- Q2 pad D1: /DRAIN_1 -> /DRAIN_2
- Q2 pad D2: /DRAIN_2 -> /DRAIN_1
- Q2 pad G1: /PWM_1 -> /PWM_2
- Q2 pad G2: /PWM_2 -> /PWM_1
- R1 pad 1: Net-(Q1-Pad3) -> Net-(Q1-PadS)
- U1 pad 1: Net-(Q1-Pad3) -> Net-(Q1-PadS)
Routing:
- net Net-(Q1-PadS): track 0.00 -> 18.3 mm
- net /SENSE: track 42.6 -> 59.5 mm
- net GND: track 6.16 -> 21.3 mm, vias 11 -> 22
- net /PWM_5: track 44.8 -> 53.3 mm
- net /PWM_1: track 26.9 -> 34.4 mm
- net Net-(Q1-Pad3): track 7.21 -> 0.00 mm
- net /DRAIN_7: track 0.00 -> 7.16 mm
- net /DRAIN_5: track 0.00 -> 6.97 mm
- net /RESET: track 25.4 -> 18.5 mm
- net /DRAIN_6: track 0.00 -> 6.12 mm
- net /DRAIN_8: track 0.00 -> 5.87 mm, vias 2 -> 0
- net +12V: track 52.0 -> 57.7 mm
- net /PWM_6: track 42.8 -> 47.6 mm
- net /PWM_3: track 19.4 -> 21.4 mm
- net /PWR_EN: track 34.7 -> 32.9 mm
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- removed copper zone on B.Cu, net /DRAIN_5
- removed copper zone on B.Cu, net /DRAIN_6
- removed copper zone on B.Cu, net /DRAIN_7
- removed copper zone on B.Cu, net /DRAIN_8

Commit message: starting rev1
Routing:
- net /DRAIN_3: track 0.00 -> 8.07 mm
- net /DRAIN_1: track 0.00 -> 7.68 mm
- net /DRAIN_4: track 0.00 -> 6.81 mm
- net /DRAIN_2: track 0.00 -> 5.78 mm
- net +12V: track 57.7 -> 52.4 mm
- net /DRAIN_8: track 5.87 -> 7.05 mm
- net /SW_A1: track 59.4 -> 60.4 mm
- net /DRAIN_7: track 7.16 -> 7.82 mm
- net /DRAIN_6: track 6.12 -> 6.74 mm
- net /PWR_EN: track 32.9 -> 33.5 mm
- removed copper zone on B.Cu, net /DRAIN_1
- removed copper zone on B.Cu, net /DRAIN_2
- removed copper zone on B.Cu, net /DRAIN_3
- removed copper zone on B.Cu, net /DRAIN_4
